Commit message: Add Laser scan to simulatiom

File: src/wro_ws/src/simulation/models/robot/robot.urdf.xacro (robot description, xacro)
@@ -3,3 +3,4 @@
   <xacro:include filename="robot_core.xacro" />
   <xacro:include filename="gazebo_control.xacro" />
+  <xacro:include filename="lidar.xacro" />
 </robot>

File: src/wro_ws/src/simulation/models/robot/robot_core.xacro (robot description, xacro)
@@ -18,5 +18,5 @@
             <box size="2 1 0.4"/>
           </geometry>
-          <material name="green" />
+          <material name="orange" />
         </visual>
         <collision>
@@ -51,5 +51,5 @@
             </friction>
           </surface>
-        <material name="white"/>
+        <material name="black"/>
       </visual>
       <xacro:inertial_cylinder mass="1.0" length="0.1" radius="0.2">
@@ -89,5 +89,5 @@
           <cylinder length="0.1" radius="0.2"/>
         </geometry>
-        <material name="white"/>
+        <material name="black"/>
       </visual>
       <xacro:inertial_cylinder mass="1.0" length="0.1" radius="0.2">
@@ -127,5 +127,5 @@
           <cylinder length="0.1" radius="0.2"/>
         </geometry>
-        <material name="white"/>
+        <material name="black"/>
       </visual>
       <xacro:inertial_cylinder mass="1.0" length="0.1" radius="0.2">
@@ -157,5 +157,5 @@
           <cylinder length="0.1" radius="0.2"/>
         </geometry>
-        <material name="white"/>
+        <material name="black"/>
       </visual>
       <xacro:inertial_cylinder mass="1.0" length="0.1" radius="0.2">
@@ -178,5 +178,5 @@
           <cylinder radius="0.04" length="0.2"/>
         </geometry>
-        <material name="white"/>
+        <material name="black"/>
       </visual>
       <xacro:inertial_cylinder mass="0.4" length="0.2" radius="0.04">
@@ -196,5 +196,5 @@
           <cylinder radius="0.04" length="0.2"/>
         </geometry>
-        <material name="white"/>
+        <material name="black"/>
       </visual>
       <xacro:inertial_cylinder mass="0.4" length="0.2" radius="0.04">
