Commit message: Add lidar

File: src/wro_ws/src/robot_description/urdf/lidar.xacro (robot description, xacro)
@@ -4,19 +4,19 @@
         <parent link="base_link"/>
         <child link="laser_frame"/>
-        <origin xyz="0 0 0.3" rpy="0 0 0"/>
+        <origin xyz="0 0 0.038" rpy="0 0 0"/>
     </joint>
     <link name="laser_frame">
         <collision>
             <geometry>
-            <cylinder length="0.1" radius="0.2"/>
+            <cylinder length="0.02" radius="0.04"/>
             </geometry>
         </collision>
         <visual>
             <geometry>
-            <cylinder length="0.1" radius="0.2"/>
+            <cylinder length="0.02" radius="0.04"/>
             </geometry>
             <material name="green"/>
         </visual>
-        <xacro:inertial_cylinder mass="1.0" length="0.1" radius="0.2">
+        <xacro:inertial_cylinder mass="1.0" length="0.02" radius="0.04">
             <origin xyz="0 0 0" rpy="0 0 0"/>
         </xacro:inertial_cylinder>

File: src/wro_ws/src/robot_description/urdf/robot.urdf.xacro (robot description, xacro)
@@ -3,5 +3,5 @@
   <xacro:include filename="robot_core.xacro" />
   <xacro:include filename="gazebo_control.xacro" />
-  <!-- <xacro:include filename="lidar.xacro" /> -->
+  <xacro:include filename="lidar.xacro" />
   <!-- <xacro:include filename="camera.xacro" /> -->
   <!-- <xacro:include filename="depth_camera.xacro" /> -->
