Commit message: Set up ros2 control and write plugin for ackerman steering

File: src/wro_ws/src/robot_description/urdf/colors.xacro (robot description, xacro)
@@ -16,3 +16,6 @@
         <color rgba="1 0.3 0.1 1"/>
     </material>
+    <material name="invisible">
+        <color rgba="0.0 0.0 0.0 0.0"/>
+    </material>
 </robot>

File: src/wro_ws/src/robot_description/urdf/robot.urdf.xacro (robot description, xacro)
@@ -1,7 +1,10 @@
 <?xml version="1.0"?>
 <robot name="my_robot" xmlns:xacro="http://www.ros.org/wiki/xacro">
-  <xacro:include filename="robot_core.xacro" />
-  <xacro:include filename="gazebo_control.xacro" />
-  <xacro:include filename="lidar.xacro" />
+  <!-- <xacro:include filename="robot_core.xacro" /> -->
+  <xacro:include filename="physical_robot_core.xacro" />
+  <!-- <xacro:include filename="gazebo_control.xacro" /> -->
+  <!-- <xacro:include filename="ros2_control_ack.xacro" /> -->
+  <xacro:include filename="ros2_control_bic.xacro" />
+  <!-- <xacro:include filename="lidar.xacro" /> -->
   <!-- <xacro:include filename="camera.xacro" /> -->
   <!-- <xacro:include filename="depth_camera.xacro" /> -->

File: src/wro_ws/src/robot_description/urdf/robot_core.xacro (robot description, xacro)
@@ -14,11 +14,4 @@
     <xacro:property name="wheel_zoff" value="0.03"/>
     <xacro:property name="wheel_xoff" value="0.09"/>
-    <link name="base_footprint" />
-    <joint name="base_joint" type="fixed">
-        <parent link="base_footprint" />
-        <child link="base_link" />
-        <origin xyz="0 0 ${(wheel_radius+wheel_zoff)}" rpy="0 0 0" />
-    </joint>
-    <!-- Chassis -->
     <link name="base_link">
         <visual>

File: src/wro_ws/src/simulation/models/robot/colors.xacro (robot description, xacro)
@@ -16,3 +16,6 @@
         <color rgba="1 0.3 0.1 1"/>
     </material>
+    <material name="invisible">
+        <color rgba="0.0 0.0 0.0 0.0"/>
+    </material>
 </robot>

File: src/wro_ws/src/simulation/models/robot/gazebo_control.xacro (robot description, xacro)
@@ -30,5 +30,5 @@
         <!-- Frame -->
         <odometry_frame>odom</odometry_frame>
-        <robot_base_frame>base_footprint</robot_base_frame>
+        <robot_base_frame>base_link</robot_base_frame>
       </plugin>
     </gazebo>

File: src/wro_ws/src/simulation/models/robot/robot.urdf.xacro (robot description, xacro)
@@ -2,5 +2,7 @@
 <robot name="my_robot" xmlns:xacro="http://www.ros.org/wiki/xacro">
   <xacro:include filename="robot_core.xacro" />
-  <xacro:include filename="gazebo_control.xacro" />
+  <!-- <xacro:include filename="gazebo_control.xacro" /> -->
+  <!-- <xacro:include filename="ros2_control.xacro" /> -->
+  <xacro:include filename="ros2_control_bic.xacro" />
   <xacro:include filename="lidar.xacro" />
   <!-- <xacro:include filename="camera.xacro" /> -->

File: src/wro_ws/src/simulation/models/robot/robot_core.xacro (robot description, xacro)
@@ -3,10 +3,4 @@
     <xacro:include filename="colors.xacro" />
     <xacro:include filename="inertial_macros.xacro" />
-    <link name="base_footprint" />
-    <joint name="base_joint" type="fixed">
-        <parent link="base_footprint" />
-        <child link="base_link" />
-        <origin xyz="0 0 0.3" rpy="0 0 0" />
-    </joint>
     <link name='base_link'>
         <xacro:inertial_box mass="20" x="2" y="1" z="0.4">
@@ -30,4 +24,31 @@
         <material>Gazebo/Orange</material>
     </gazebo>
+    <link name="virtual_rear_wheel">
+      <visual>
+        <origin xyz="0 0 0" rpy="0 1.5708 1.5708" />
+        <geometry>
+          <cylinder length="0.01" radius="0.2"/>
+        </geometry>
+        <material name="invisible"/>
+      </visual>
+      <collision>
+        <origin xyz="0 0 0" rpy="0 1.5708 1.5708" />
+        <geometry>
+          <cylinder length="0.01" radius="0.2"/>
+        </geometry>
+        <material name="invisible"/>
+      </collision>
+      <xacro:inertial_cylinder mass="1.0" length="0.01" radius="0.2">
+            <origin xyz="0 0 0" rpy="0 1.5708 1.5708"/>
+      </xacro:inertial_cylinder>
+    </link>
+    <joint name="virtual_rear_wheel_joint" type="continuous">
+      <parent link="base_link"/>
+      <child link="virtual_rear_wheel"/>
+      <origin xyz="-0.7 0 -0.1" rpy="0 0 0"/>
+      <axis xyz="0 1 0" rpy="0 0 0" />
+      <limit effort="100.0" velocity="100.0"/>
+      <dynamics damping="0.2"/>
+    </joint>
     <link name="right_wheel_rear">
       <collision>
@@ -36,6 +57,134 @@
           <cylinder length="0.1" radius="0.2"/>
         </geometry>
-      </collision>
-      <visual>
+        <surface>
+          <friction>
+            <ode>
+              <mu>2.0</mu>
+              <mu2>2.0</mu2>
+              <fdir1>0 0 1</fdir1>
+            </ode>
+          </friction>
+        </surface>
+      </collision>
+      <visual>
+        <origin xyz="0 0 0" rpy="0 1.5708 1.5708" />
+        <geometry>
+          <cylinder length="0.1" radius="0.2"/>
+        </geometry>
+        <material name="black"/>
+      </visual>
+      <xacro:inertial_cylinder mass="1.0" length="0.1" radius="0.2">
+            <origin xyz="0 0 0" rpy="0 1.5708 1.5708"/>
+      </xacro:inertial_cylinder>
+    </link>
+    <gazebo reference="right_wheel_rear">
+      <material>Gazebo/Black</material>
+    </gazebo>
+    <joint name="base_right_wheel_rear_joint" type="continuous">
+      <parent link="base_link"/>
+      <child link="right_wheel_rear"/>
+      <origin xyz="-0.7 0.52 -0.1" rpy="0 0 0" />
+      <axis xyz="0 1 0" rpy="0 0 0" />
+      <!-- <limit effort="100" velocity="10"/>
+      <dynamics damping="0.1" friction="0.2"/>  -->
+      <limit effort="100.0" velocity="100.0"/>
+      <dynamics damping="0.2" />
+      <!-- <mimic joint="virtual_rear_wheel_joint" multiplier="1.0" offset="0.0"/> -->
+    </joint>
+    <link name="left_wheel_rear">
+      <collision>
+        <origin xyz="0 0 0" rpy="0 1.5708 1.5708" />
+        <geometry>
+          <cylinder length="0.1" radius="0.2"/>
+        </geometry>
+        <surface>
+          <friction>
+            <ode>
+              <mu>2.0</mu>
+              <mu2>2.0</mu2>
+              <fdir1>0 0 1</fdir1>
+            </ode>
+          </friction>
+        </surface>
+      </collision>
+      <visual>
+        <origin xyz="0 0 0" rpy="0 1.5708 1.5708" />
+        <geometry>
+          <cylinder length="0.1" radius="0.2"/>
+        </geometry>
+        <material name="black"/>
+      </visual>
+      <xacro:inertial_cylinder mass="1.0" length="0.1" radius="0.2">
+            <origin xyz="0 0 0" rpy="0 1.5708 1.5708"/>
+      </xacro:inertial_cylinder>
+    </link>
+    <gazebo reference="left_wheel_rear">
+      <material>Gazebo/Black</material>
+    </gazebo>
+    <joint name="base_left_wheel_rear_joint" type="continuous">
+      <parent link="base_link"/>
+      <child link="left_wheel_rear"/>
+      <origin xyz="-0.7 -0.52 -0.1" rpy="0 0 0" />
+      <axis xyz="0 1 0" rpy="0 0 0" />
+      <!-- <limit effort="100" velocity="10"/>
+      <dynamics damping="0.1" friction="0.2"/> -->
+      <limit effort="100.0" velocity="100.0"/>
+      <dynamics damping="0.2" />
+      <!-- <mimic joint="virtual_rear_wheel_joint" multiplier="1.0" offset="0.0"/> -->
+    </joint>
+    <link name="virtual_front_wheel">
+      <visual>
+        <origin xyz="0 0 0" rpy="0 1.5708 1.5708" />
+        <geometry>
+          <cylinder length="0.01" radius="0.2"/>
+        </geometry>
+        <material name="invisible"/>
+      </visual>
+      <collision>
+        <origin xyz="0 0 0" rpy="0 1.5708 1.5708" />
+        <geometry>
+          <cylinder length="0.01" radius="0.2"/>
+        </geometry>
+        <material name="invisible"/>
+      </collision>
+      <xacro:inertial_cylinder mass="1.0" length="0.01" radius="0.2">
+            <origin xyz="0 0 0" rpy="0 1.5708 1.5708"/>
+      </xacro:inertial_cylinder>
+    </link>
+    <link name="virtual_steer">
+      <visual>
+        <origin xyz="0 0 0" rpy="0 0 0" />
+        <geometry>
+          <cylinder length="0.02" radius="0.04"/>
+        </geometry>
+        <material name="invisible"/>
+      </visual>
+      <collision>
+        <origin xyz="0 0 0" rpy="0 0 0"/>
+        <geometry>
+          <cylinder radius="0.04" length="0.02"/>
+        </geometry>
+      </collision>
+      <xacro:inertial_cylinder mass="0.4" length="0.02" radius="0.04">
+        <origin xyz="0 0 0" rpy="0 0 0"/>
+      </xacro:inertial_cylinder>
+    </link>
+    <joint name="virtual_steer_joint" type="revolute">
+      <parent link="base_link"/>
+      <child link="virtual_steer"/>
+      <origin xyz="0.7 0 -0.1" rpy="0 0 0"/>
+      <axis xyz="0 0 1" rpy="0 0 0" />
+      <limit lower="-0.6" upper="0.6" velocity="25.0" effort="25.0"/>
+    </joint>
+    <joint name="virtual_front_wheel_joint" type="continuous">
+      <parent link="virtual_steer"/>
+      <child link="virtual_front_wheel"/>
+      <origin xyz="0 0 0" rpy="0 0 0"/>
+      <axis xyz="0 1 0" rpy="0 0 0" />
+      <limit effort="100" velocity="100"/>
+      <dynamics damping="0.1" friction="0.2"/>
+    </joint>
+    <link name="right_wheel_front">
+      <collision>
         <origin xyz="0 0 0" rpy="0 1.5708 1.5708" />
         <geometry>
@@ -51,74 +200,4 @@
             </friction>
           </surface>
-        <material name="black"/>
-      </visual>
-      <xacro:inertial_cylinder mass="1.0" length="0.1" radius="0.2">
-            <origin xyz="0 0 0" rpy="0 1.5708 1.5708"/>
-      </xacro:inertial_cylinder>
-    </link>
-    <gazebo reference="right_wheel_rear">
-      <material>Gazebo/Black</material>
-    </gazebo>
-    <joint name="base_right_wheel_rear_joint" type="continuous">
-      <parent link="base_link"/>
-      <child link="right_wheel_rear"/>
-      <origin xyz="-0.7 0.52 -0.1" rpy="0 0 0" />
-      <axis xyz="0 1 0" rpy="0 0 0" />
-      <limit effort="100" velocity="10"/>
-      <dynamics damping="0.1" friction="0.2"/>
-    </joint>
-    <link name="left_wheel_rear">
-      <collision>
-        <origin xyz="0 0 0" rpy="0 1.5708 1.5708" />
-        <geometry>
-          <cylinder length="0.1" radius="0.2"/>
-        </geometry>
-          <surface>
-            <friction>
-              <ode>
-                <mu>2.0</mu>
-                <mu2>2.0</mu2>
-                <fdir1>0 0 1</fdir1>
-              </ode>
-            </friction>
-          </surface>
-      </collision>
-      <visual>
-        <origin xyz="0 0 0" rpy="0 1.5708 1.5708" />
-        <geometry>
-          <cylinder length="0.1" radius="0.2"/>
-        </geometry>
-        <material name="black"/>
-      </visual>
-      <xacro:inertial_cylinder mass="1.0" length="0.1" radius="0.2">
-            <origin xyz="0 0 0" rpy="0 1.5708 1.5708"/>
-      </xacro:inertial_cylinder>
-    </link>
-    <gazebo reference="left_wheel_rear">
-      <material>Gazebo/Black</material>
-    </gazebo>
-    <joint name="base_left_wheel_rear_joint" type="continuous">
-      <parent link="base_link"/>
-      <child link="left_wheel_rear"/>
-      <origin xyz="-0.7 -0.52 -0.1" rpy="0 0 0" />
-      <axis xyz="0 1 0" rpy="0 0 0" />
-      <limit effort="100" velocity="10"/>
-      <dynamics damping="0.1" friction="0.2"/>
-    </joint>
-    <link name="right_wheel_front">
-      <collision>
-        <origin xyz="0 0 0" rpy="0 1.5708 1.5708" />
-        <geometry>
-          <cylinder length="0.1" radius="0.2"/>
-        </geometry>
-          <surface>
-            <friction>
-              <ode>
-                <mu>2.0</mu>
-                <mu2>2.0</mu2>
-                <fdir1>0 0 1</fdir1>
-              </ode>
-            </friction>
-          </surface>
       </collision>
       <visual>
@@ -208,4 +287,5 @@
       <axis xyz="0 0 1" rpy="0 0 0"/>
       <limit lower="-0.6" upper="0.6" velocity="1.0" effort="25"/>
+      <!-- <mimic joint="virtual_steer_joint" multiplier="1.0" offset="0.0"/> -->
     </joint>
     <joint name="front_right_wheel_steering_joint" type="revolute">
@@ -215,4 +295,5 @@
       <axis xyz="0 0 1" rpy="0 0 0"/>
       <limit lower="-0.6" upper="0.6" velocity="1.0" effort="25"/>
+      <!-- <mimic joint="virtual_steer_joint" multiplier="1.0" offset="0.0"/> -->
     </joint>
     <joint name="front_left_wheel_joint" type="continuous">
@@ -223,4 +304,5 @@
       <limit effort="100" velocity="10"/>
       <dynamics damping="0.1" friction="0.2"/>
+      <!-- <mimic joint="virtual_front_wheel_joint" multiplier="1.0" offset="0.0"/> -->
     </joint>
     <joint name="front_right_wheel_joint" type="continuous">
@@ -231,4 +313,5 @@
       <limit effort="100" velocity="10"/>
       <dynamics damping="0.1" friction="0.2"/>
+      <!-- <mimic joint="virtual_front_wheel_joint" multiplier="1.0" offset="0.0"/> -->
     </joint>
 </robot>
