Commit message: Add default maps

File: src/wro_ws/src/robot_description/urdf/physical_robot_core.xacro (robot description, xacro)
@@ -36,4 +36,11 @@
       </inertial>
     </link>
+    <joint name="base_footprint_joint" type="fixed">
+        <parent link="base_link"/>
+        <child link="base_footprint"/>
+        <origin xyz="0 0 0" rpy="0 0 0"/>
+    </joint>
+    <link name="base_footprint">
+    </link>
     <!-- rear wheels -->
     <!-- virtual rear wheel -->
