Commit message: Add accurate robot description

File: src/wro_ws/src/robot_description/urdf/depth_camera.xacro (robot description, xacro)
@@ -4,10 +4,10 @@
         <parent link="base_link"/>
         <child link="camera_link"/>
-        <origin xyz="1 0 0.1" rpy="0 0 0"/>
+        <origin xyz="0.1 0 0.01" rpy="0 0 0"/>
     </joint>
     <link name="camera_link">
         <visual>
             <geometry>
-                <box size="0.1 0.15 0.15"/>
+                <box size="0.006 0.02 0.02"/>
             </geometry>
             <material name="green"/>
@@ -22,5 +22,5 @@
     <gazebo reference="camera_link">
         <material>Gazebo/Green</material>
-        <gravity>true</gravity>
+        <!-- <gravity>true</gravity> -->
         <sensor name="camera" type="depth">
             <pose>0 0 0 0 0 0</pose>
@@ -47,5 +47,5 @@
         <!-- <sensor name="imu_sensor" type="imu">
             <always_on>true</always_on>
-            <update_rate>1</update_rate>
+            <update_rate>100</update_rate>
             <visualize>true</visualize>
             <topic>__default_topic__</topic>
@@ -61,70 +61,69 @@
             <pose>0 0 0 0 0 0</pose>
         </sensor> -->
-        <sensor name="imu_sensor" type="imu">
-            <plugin filename="libgazebo_ros_imu_sensor.so" name="imu">
+        <!-- <sensor name="imu_sensor" type="imu">
+            <plugin filename="libgazebo_ros_imu_sensor.so" name="imu_plugin">
                 <ros>
-                    <!-- <namespace>/demo</namespace> -->
                     <remapping>~/out:=imu</remapping>
                 </ros>
                 <initial_orientation_as_reference>false</initial_orientation_as_reference>
-            </plugin>
-            <always_on>true</always_on>
-            <update_rate>100</update_rate>
-            <visualize>true</visualize>
-            <imu>
+                </plugin>
+                <always_on>true</always_on>
+                <update_rate>100</update_rate>
+                <visualize>true</visualize>
+                <imu>
                 <angular_velocity>
                     <x>
-                        <noise type="gaussian">
-                            <mean>0.0</mean>
-                            <stddev>2e-4</stddev>
-                            <bias_mean>0.0000075</bias_mean>
-                            <bias_stddev>0.0000008</bias_stddev>
-                        </noise>
+                    <noise type="gaussian">
+                        <mean>0.0</mean>
+                        <stddev>2e-4</stddev>
+                        <bias_mean>0.0000075</bias_mean>
+                        <bias_stddev>0.0000008</bias_stddev>
+                    </noise>
                     </x>
                     <y>
-                        <noise type="gaussian">
-                            <mean>0.0</mean>
-                            <stddev>2e-4</stddev>
-                            <bias_mean>0.0000075</bias_mean>
-                            <bias_stddev>0.0000008</bias_stddev>
-                        </noise>
+                    <noise type="gaussian">
+                        <mean>0.0</mean>
+                        <stddev>2e-4</stddev>
+                        <bias_mean>0.0000075</bias_mean>
+                        <bias_stddev>0.0000008</bias_stddev>
+                    </noise>
                     </y>
                     <z>
-                        <noise type="gaussian">
-                            <mean>0.0</mean>
-                            <stddev>2e-4</stddev>
-                            <bias_mean>0.0000075</bias_mean>
-                            <bias_stddev>0.0000008</bias_stddev>
-                        </noise>
+                    <noise type="gaussian">
+                        <mean>0.0</mean>
+                        <stddev>2e-4</stddev>
+                        <bias_mean>0.0000075</bias_mean>
+                        <bias_stddev>0.0000008</bias_stddev>
+                    </noise>
                     </z>
                 </angular_velocity>
                 <linear_acceleration>
                     <x>
-                        <noise type="gaussian">
-                            <mean>0.0</mean>
-                            <stddev>1.7e-2</stddev>
-                            <bias_mean>0.1</bias_mean>
-                            <bias_stddev>0.001</bias_stddev>
-                        </noise>
+                    <noise type="gaussian">
+                        <mean>0.0</mean>
+                        <stddev>1.7e-2</stddev>
+                        <bias_mean>0.1</bias_mean>
+                        <bias_stddev>0.001</bias_stddev>
+                    </noise>
                     </x>
                     <y>
-                        <noise type="gaussian">
-                            <mean>0.0</mean>
-                            <stddev>1.7e-2</stddev>
-                            <bias_mean>0.1</bias_mean>
-                            <bias_stddev>0.001</bias_stddev>
-                        </noise>
+                    <noise type="gaussian">
+                        <mean>0.0</mean>
+                        <stddev>1.7e-2</stddev>
+                        <bias_mean>0.1</bias_mean>
+                        <bias_stddev>0.001</bias_stddev>
+                    </noise>
                     </y>
                     <z>
-                        <noise type="gaussian">
-                            <mean>0.0</mean>
-                            <stddev>1.7e-2</stddev>
-                            <bias_mean>0.1</bias_mean>
-                            <bias_stddev>0.001</bias_stddev>
-                        </noise>
+                    <noise type="gaussian">
+                        <mean>0.0</mean>
+                        <stddev>1.7e-2</stddev>
+                        <bias_mean>0.1</bias_mean>
+                        <bias_stddev>0.001</bias_stddev>
+                    </noise>
                     </z>
                 </linear_acceleration>
             </imu>
-        </sensor>
+        </sensor> -->
     </gazebo>
 </robot>

File: src/wro_ws/src/robot_description/urdf/robot_core_2.xacro (robot description, xacro)
@@ -1,19 +1,6 @@
 <?xml version="1.0"?>
-<robot name="my_robot" xmlns:xacro="http://www.ros.org/wiki/xacro">
-    <material name="grey">
-        <color rgba="0.7 0.7 0.7 1"/>
-    </material>
-    <material name="green">
-        <color rgba="0 0.6 0 1"/>
-    </material>
-    <material name="white">
-        <color rgba="1 1 1 1"/>
-    </material>
-    <material name="black">
-        <color rgba="0 0 0 1"/>
-    </material>
-    <material name="orange">
-        <color rgba="1 0.3 0.1 1"/>
-    </material>
+<robot xmlns:xacro="http://www.ros.org/wiki/xacro">
+    <xacro:include filename="colors.xacro" />
+    <xacro:include filename="inertial_macros.xacro" />
     <link name="base_footprint" />
     <joint name="base_joint" type="fixed">
@@ -23,9 +10,7 @@
     </joint>
     <link name='base_link'>
-        <inertial>
-          <mass value="1.14"/>
-          <origin xyz="0 0 0.05" rpy="0 0 0"/>
-          <inertia ixx="0.13" ixy="0" ixz="0" iyy="0.4" iyz="0" izz="0.48"/>
-        </inertial>
+        <xacro:inertial_box mass="20" x="2" y="1" z="0.4">
+            <origin xyz="0 0 0.05" rpy="0 0 0"/>
+        </xacro:inertial_box>
         <visual>
           <origin xyz="0 0 0.05" rpy="0 0 0"/>
@@ -33,10 +18,10 @@
             <box size="2 1 0.4"/>
           </geometry>
-          <material name="green" />
+          <material name="orange" />
         </visual>
         <collision>
           <origin xyz="0 0 0.05" rpy="0 0 0"/>
           <geometry>
-                <box size="2 1 0.4"/>
+            <box size="2 1 0.4"/>
           </geometry>
         </collision>
@@ -49,22 +34,29 @@
         <origin xyz="0 0 0" rpy="0 1.5708 1.5708" />
         <geometry>
-        <cylinder length="0.1" radius="0.2"/>
-        </geometry>
-      </collision>
-      <visual>
-        <origin xyz="0 0 0" rpy="0 1.5708 1.5708" />
-        <geometry>
-        <cylinder length="0.1" radius="0.2"/>
-        </geometry>
-        <material name="white"/>
-      </visual>
-      <inertial>
-        <origin xyz="0 0 0" rpy="0 1.5708 1.5708" />
-        <mass value="0.2"/>
-        <inertia ixx="0.15" ixy="0" ixz="0" iyy="0.15" iyz="0" izz="0.125"/>
-      </inertial>
+          <cylinder length="0.1" radius="0.2"/>
+        </geometry>
+        <surface>
+          <friction>
+            <ode>
+              <mu>2.0</mu>
+              <mu2>2.0</mu2>
+              <fdir1>0 0 1</fdir1>
+            </ode>
+          </friction>
+        </surface>
+      </collision>
+      <visual>
+        <origin xyz="0 0 0" rpy="0 1.5708 1.5708" />
+        <geometry>
+          <cylinder length="0.1" radius="0.2"/>
+        </geometry>
+        <material name="black"/>
+      </visual>
+      <xacro:inertial_cylinder mass="1.0" length="0.1" radius="0.2">
+            <origin xyz="0 0 0" rpy="0 1.5708 1.5708"/>
+      </xacro:inertial_cylinder>
     </link>
     <gazebo reference="right_wheel_rear">
-        <material>Gazebo/Black</material>
+      <material>Gazebo/Black</material>
     </gazebo>
     <joint name="base_right_wheel_rear_joint" type="continuous">
@@ -74,5 +66,5 @@
       <axis xyz="0 1 0" rpy="0 0 0" />
       <limit effort="100" velocity="10"/>
-      <dynamics damping="0.0" friction="0.0"/>
+      <dynamics damping="0.1" friction="0.2"/>
     </joint>
     <link name="left_wheel_rear">
@@ -82,20 +74,27 @@
           <cylinder length="0.1" radius="0.2"/>
         </geometry>
-      </collision>
-      <visual>
-        <origin xyz="0 0 0" rpy="0 1.5708 1.5708" />
-        <geometry>
-          <cylinder length="0.1" radius="0.2"/>
-        </geometry>
-        <material name="white"/>
-      </visual>
-      <inertial>
-        <origin xyz="0 0 0" rpy="0 1.5708 1.5708" />
-        <mass value="0.2"/>
-        <inertia ixx="0.15" ixy="0" ixz="0" iyy="0.15" iyz="0" izz="0.125"/>
-      </inertial>
+          <surface>
+            <friction>
+              <ode>
+                <mu>2.0</mu>
+                <mu2>2.0</mu2>
+                <fdir1>0 0 1</fdir1>
+              </ode>
+            </friction>
+          </surface>
+      </collision>
+      <visual>
+        <origin xyz="0 0 0" rpy="0 1.5708 1.5708" />
+        <geometry>
+          <cylinder length="0.1" radius="0.2"/>
+        </geometry>
+        <material name="black"/>
+      </visual>
+      <xacro:inertial_cylinder mass="1.0" length="0.1" radius="0.2">
+            <origin xyz="0 0 0" rpy="0 1.5708 1.5708"/>
+      </xacro:inertial_cylinder>
     </link>
     <gazebo reference="left_wheel_rear">
-        <material>Gazebo/Black</material>
+      <material>Gazebo/Black</material>
     </gazebo>
     <joint name="base_left_wheel_rear_joint" type="continuous">
@@ -105,5 +104,5 @@
       <axis xyz="0 1 0" rpy="0 0 0" />
       <limit effort="100" velocity="10"/>
-      <dynamics damping="0.0" friction="0.0"/>
+      <dynamics damping="0.1" friction="0.2"/>
     </joint>
     <link name="right_wheel_front">
@@ -113,20 +112,27 @@
           <cylinder length="0.1" radius="0.2"/>
         </geometry>
-      </collision>
-      <visual>
-        <origin xyz="0 0 0" rpy="0 1.5708 1.5708" />
-        <geometry>
-          <cylinder length="0.1" radius="0.2"/>
-        </geometry>
-        <material name="white"/>
-      </visual>
-      <inertial>
-        <origin xyz="0 0 0" rpy="0 1.5708 1.5708" />
-        <mass value="0.2"/>
-        <inertia ixx="0.15" ixy="0" ixz="0" iyy="0.15" iyz="0" izz="0.125"/>
-      </inertial>
+          <surface>
+            <friction>
+              <ode>
+                <mu>2.0</mu>
+                <mu2>2.0</mu2>
+                <fdir1>0 0 1</fdir1>
+              </ode>
+            </friction>
+          </surface>
+      </collision>
+      <visual>
+        <origin xyz="0 0 0" rpy="0 1.5708 1.5708" />
+        <geometry>
+          <cylinder length="0.1" radius="0.2"/>
+        </geometry>
+        <material name="black"/>
+      </visual>
+      <xacro:inertial_cylinder mass="1.0" length="0.1" radius="0.2">
+        <origin xyz="0 0 0" rpy="0 1.5708 1.5708"/>
+      </xacro:inertial_cylinder>
     </link>
     <gazebo reference="right_wheel_front">
-        <material>Gazebo/Black</material>
+      <material>Gazebo/Black</material>
     </gazebo>
     <link name="left_wheel_front">
@@ -136,46 +142,28 @@
           <cylinder length="0.1" radius="0.2"/>
         </geometry>
-      </collision>
-      <visual>
-        <origin xyz="0 0 0" rpy="0 1.5708 1.5708" />
-        <geometry>
-          <cylinder length="0.1" radius="0.2"/>
-        </geometry>
-        <material name="white"/>
-      </visual>
-      <inertial>
-        <origin xyz="0 0 0" rpy="0 1.5708 1.5708" />
-        <mass value="0.2"/>
-        <inertia ixx="0.15" ixy="0" ixz="0" iyy="0.15" iyz="0" izz="0.125"/>
-      </inertial>
+          <surface>
+            <friction>
+              <ode>
+                <mu>2.0</mu>
+                <mu2>4.0</mu2>
+                <fdir1>0 0 1</fdir1>
+              </ode>
+            </friction>
+          </surface>
+      </collision>
+      <visual>
+        <origin xyz="0 0 0" rpy="0 1.5708 1.5708" />
+        <geometry>
+          <cylinder length="0.1" radius="0.2"/>
+        </geometry>
+        <material name="black"/>
+      </visual>
+      <xacro:inertial_cylinder mass="1.0" length="0.1" radius="0.2">
+          <origin xyz="0 0 0" rpy="0 1.5708 1.5708"/>
+      </xacro:inertial_cylinder>
     </link>
     <gazebo reference="left_wheel_front">
-        <material>Gazebo/Black</material>
-    </gazebo>
-    <!-- <link name="lidar_link">
-      <collision>
-        <origin xyz="0 0 0" rpy="0 0 0"/>
-        <geometry>
-          <cylinder radius="0.13" length="0.1"/>
-        </geometry>
-      </collision>
-      <visual>
-        <origin xyz="0 0 0" rpy="0 0 0"/>
-        <geometry>
-          <cylinder radius="0.13" length="0.1"/>
-        </geometry>
-        <material name="white"/>
-      </visual>
-      <inertial>
-        <origin xyz="0 0 0" rpy="0 0 0"/>
-        <mass value="0.1"/>
-        <inertia ixx="0.0001" ixy="0" ixz="0" iyy="0.0001" iyz="0" izz="0.0001"/>
-      </inertial>
-    </link>
-    <joint name="base_lidar_joint" type="fixed">
-      <parent link="base_link"/>
-      <child link="lidar_link"/>
-      <origin xyz="0 0 0.4" rpy="0 0 0"/>
-    </joint> -->
+      <material>Gazebo/Black</material>
+    </gazebo>
     <link name="front_left_wheel_steering_link">
       <collision>
@@ -190,11 +178,9 @@
           <cylinder radius="0.04" length="0.2"/>
         </geometry>
-        <material name="white"/>
-      </visual>
-      <inertial>
-        <origin xyz="0 0 0" rpy="0 0 0"/>
-        <mass value="0.5"/>
-        <inertia ixx="0.0153" ixy="0" ixz="0" iyy="0.025" iyz="0" izz="0.0153"/>
-      </inertial>
+        <material name="black"/>
+      </visual>
+      <xacro:inertial_cylinder mass="0.4" length="0.2" radius="0.04">
+        <origin xyz="0 0 0" rpy="0 0 0"/>
+      </xacro:inertial_cylinder>
     </link>
     <link name="front_right_wheel_steering_link">
@@ -210,11 +196,9 @@
           <cylinder radius="0.04" length="0.2"/>
         </geometry>
-        <material name="white"/>
-      </visual>
-      <inertial>
-        <origin xyz="0 0 0" rpy="0 0 0"/>
-        <mass value="0.5"/>
-        <inertia ixx="0.0153" ixy="0" ixz="0" iyy="0.025" iyz="0" izz="0.0153"/>
-      </inertial>
+        <material name="black"/>
+      </visual>
+      <xacro:inertial_cylinder mass="0.4" length="0.2" radius="0.04">
+        <origin xyz="0 0 0" rpy="0 0 0"/>
+      </xacro:inertial_cylinder>
     </link>
     <joint name="front_left_wheel_steering_joint" type="revolute">
@@ -238,5 +222,5 @@
       <axis xyz="0 1 0" rpy="0 0 0"/>
       <limit effort="100" velocity="10"/>
-      <dynamics damping="0.0" friction="0.0"/>
+      <dynamics damping="0.1" friction="0.2"/>
     </joint>
     <joint name="front_right_wheel_joint" type="continuous">
@@ -246,34 +230,5 @@
       <axis xyz="0 1 0" rpy="0 0 0"/>
       <limit effort="100" velocity="10"/>
-      <dynamics damping="0.0" friction="0.0"/>
-    </joint>
-    <gazebo>
-      <plugin name="gazebo_ros_ackermann_drive" filename="libgazebo_ros_ackermann_drive.so">
-        <update_rate>100.0</update_rate>
-        <!-- Parts info -->
-        <front_left_joint>front_left_wheel_joint</front_left_joint>
-        <front_right_joint>front_right_wheel_joint</front_right_joint>
-        <rear_left_joint>base_left_wheel_rear_joint</rear_left_joint>
-        <rear_right_joint>base_right_wheel_rear_joint</rear_right_joint>
-        <left_steering_joint>front_left_wheel_steering_joint</left_steering_joint>
-        <right_steering_joint>front_right_wheel_steering_joint</right_steering_joint>
-        <max_steer>0.6458</max_steer>
-        <max_steering_angle>7.85</max_steering_angle>
-        <max_speed>20</max_speed>
-        <!-- PID tuning -->
-        <left_steering_pid_gain>1500 0 1</left_steering_pid_gain>
-        <left_steering_i_range>0 0</left_steering_i_range>
-        <right_steering_pid_gain>1500 0 1</right_steering_pid_gain>
-        <right_steering_i_range>0 0</right_steering_i_range>
-        <linear_velocity_pid_gain>1000 0 1</linear_velocity_pid_gain>
-        <linear_velocity_i_range>0 0</linear_velocity_i_range>
-        <!-- Output -->
-        <publish_odom>true</publish_odom>
-        <publish_odom_tf>true</publish_odom_tf>
-        <publish_wheel_tf>true</publish_wheel_tf>
-        <publish_distance>true</publish_distance>
-        <odometry_frame>odom</odometry_frame>
-        <robot_base_frame>base_footprint</robot_base_frame>
-      </plugin>
-  </gazebo>
+      <dynamics damping="0.1" friction="0.2"/>
+    </joint>
 </robot>

Commit message: Fix plugin to publish state of traction wheel position

File: src/wro_ws/src/robot_description/urdf/depth_camera.xacro (robot description, xacro)
@@ -4,5 +4,5 @@
         <parent link="base_link"/>
         <child link="camera_link"/>
-        <origin xyz="0.1 0 0.01" rpy="0 0 0"/>
+        <origin xyz="0.128 0 0" rpy="0 0 0"/>
     </joint>
     <link name="camera_link">

File: src/wro_ws/src/robot_description/urdf/physical_robot_core.xacro (robot description, xacro)
@@ -51,5 +51,5 @@
       <child link="virtual_rear_wheel"/>
       <origin xyz="-${wheelbase/2} 0 -${base_height/2}" rpy="0 0 ${PI/2}"/>
-      <axis xyz="1 0 0"/>
+      <axis xyz="1 0 0" rpy="0 0 0"/>
       <limit effort="100.0" velocity="100.0"/>
       <dynamics damping="0.2"/>
@@ -83,5 +83,5 @@
       <child link="rear_right_wheel"/>
       <origin xyz="-${wheelbase/2} ${base_width/2} -${base_height/2}" rpy="0 0 ${PI/2}"/>
-      <axis xyz="1 0 0"/>
+      <axis xyz="1 0 0" rpy="0 0 0"/>
       <limit effort="100.0" velocity="100.0"/>
       <dynamics damping="0.2"/>
@@ -116,5 +116,5 @@
       <child link="rear_left_wheel" />
       <origin xyz="-${wheelbase/2} -${base_width/2} -${base_height/2}" rpy="0 0 ${PI/2}"/>
-      <axis xyz="1 0 0"/>
+      <axis xyz="1 0 0" rpy="0 0 0" />
       <limit effort="100.0" velocity="100.0"/>
       <dynamics damping="0.2"/>
@@ -137,5 +137,5 @@
       <origin xyz="${wheelbase/2} 0 -${base_height/2}" rpy="0 0 ${PI/2}"/>
       <axis xyz="0 0 1"/>
-      <limit lower="-0.4" upper="0.4" effort="100.0" velocity="0.0"/>
+      <limit lower="-0.7853" upper="0.7853" effort="100.0" velocity="100.0"/>
       <dynamics damping="0.2"/>
     </joint>
@@ -169,5 +169,5 @@
       <origin xyz="${wheelbase/2} ${base_width/2} -${base_height/2}" rpy="0 0 ${PI/2}"/>
       <axis xyz="0 0 1"/>
-      <limit lower="-0.4" upper="0.4" effort="100.0" velocity="0.0"/>
+      <limit lower="-0.7853" upper="0.7853" effort="100.0" velocity="100.0"/>
       <dynamics damping="0.2"/>
       <mimic joint="virtual_front_wheel_joint" multiplier="1.0" offset="0.0"/>
@@ -201,5 +201,5 @@
       <origin xyz="${wheelbase/2} -${base_width/2} -${base_height/2}" rpy="0 0 ${PI/2}"/>
       <axis xyz="0 0 1"/>
-      <limit lower="-0.4" upper="0.4" effort="100.0" velocity="0.0"/>
+      <limit lower="-0.7853" upper="0.7853" effort="100.0" velocity="100.0"/>
       <dynamics damping="0.2"/>
       <mimic joint="virtual_front_wheel_joint" multiplier="1.0" offset="0.0"/>

File: src/wro_ws/src/robot_description/urdf/robot.urdf.xacro (robot description, xacro)
@@ -1,11 +1,7 @@
 <?xml version="1.0"?>
 <robot name="my_robot" xmlns:xacro="http://www.ros.org/wiki/xacro">
-  <!-- <xacro:include filename="robot_core.xacro" /> -->
   <xacro:include filename="physical_robot_core.xacro" />
-  <!-- <xacro:include filename="gazebo_control.xacro" /> -->
-  <!-- <xacro:include filename="ros2_control_ack.xacro" /> -->
   <xacro:include filename="ros2_control_bic.xacro" />
-  <!-- <xacro:include filename="lidar.xacro" /> -->
-  <!-- <xacro:include filename="camera.xacro" /> -->
-  <!-- <xacro:include filename="depth_camera.xacro" /> -->
+  <xacro:include filename="lidar.xacro" />
+  <xacro:include filename="depth_camera.xacro" />
 </robot>

File: src/wro_ws/src/robot_description/urdf/ros2_control_bic.xacro (robot description, xacro)
@@ -7,5 +7,6 @@
             <param name="rear_wheel_name">virtual_rear_wheel_joint</param>
             <param name="loop_rate">30</param>
-            <param name="device">/dev/serial/by-path/platform-3610000.usb-usb-0:2.1:1.0-port0</param>
+            <!-- <param name="device">/dev/serial/by-path/platform-3610000.usb-usb-0:2.1:1.0-port0</param> -->
+            <param name="device">/dev/serial/by-path/pci-0000:00:14.0-usb-0:4:1.0-port0</param>
             <param name="baud_rate">9600</param>
             <param name="timeout_ms">1000</param>
@@ -18,4 +19,5 @@
             <command_interface name="velocity"/>
             <state_interface name="velocity"/>
+            <state_interface name="position"/>
         </joint>
     </ros2_control>
