Commit message: Set up sensor fusion between lidar and imu for odometry

File: src/wro_ws/src/robot_description/urdf/depth_camera.xacro (robot description, xacro)
@@ -20,110 +20,3 @@
     </joint>
     <link name="camera_link_optical"></link>
-    <gazebo reference="camera_link">
-        <material>Gazebo/Green</material>
-        <!-- <gravity>true</gravity> -->
-        <sensor name="camera" type="depth">
-            <pose>0 0 0 0 0 0</pose>
-            <visualize>false</visualize>
-            <update_rate>10</update_rate>
-            <camera>
-                <horizontal_fov>1.204</horizontal_fov>
-                <image>
-                    <width>640</width>
-                    <height>480</height>
-                    <format>B8G8R8</format>
-                </image>
-                <clip>
-                    <near>3</near>
-                    <far>30.0</far>
-                </clip>
-            </camera>
-            <plugin name="camera_controller" filename="libgazebo_ros_camera.so">
-                <frame_name>camera_link_optical</frame_name>
-                <min_depth>0.1</min_depth>
-                <max_depth>100</max_depth>
-            </plugin>
-        </sensor>
-        <!-- <sensor name="imu_sensor" type="imu">
-            <always_on>true</always_on>
-            <update_rate>100</update_rate>
-            <visualize>true</visualize>
-            <topic>__default_topic__</topic>
-            <plugin filename="libgazebo_ros_imu_sensor.so" name="imu_plugin">
-                <topicName>imu</topicName>
-                <bodyName>camera_link</bodyName>
-                <updateRateHZ>10.0</updateRateHZ>
-                <gaussianNoise>0.0</gaussianNoise>
-                <xyzOffset>1 0 0.1</xyzOffset>
-                <rpyOffset>0 0 0</rpyOffset>
-                <frameName>camera_link</frameName>
-            </plugin>
-            <pose>0 0 0 0 0 0</pose>
-        </sensor> -->
-        <!-- <sensor name="imu_sensor" type="imu">
-            <plugin filename="libgazebo_ros_imu_sensor.so" name="imu_plugin">
-                <ros>
-                    <remapping>~/out:=imu</remapping>
-                </ros>
-                <initial_orientation_as_reference>false</initial_orientation_as_reference>
-                </plugin>
-                <always_on>true</always_on>
-                <update_rate>100</update_rate>
-                <visualize>true</visualize>
-                <imu>
-                <angular_velocity>
-                    <x>
-                    <noise type="gaussian">
-                        <mean>0.0</mean>
-                        <stddev>2e-4</stddev>
-                        <bias_mean>0.0000075</bias_mean>
-                        <bias_stddev>0.0000008</bias_stddev>
-                    </noise>
-                    </x>
-                    <y>
-                    <noise type="gaussian">
-                        <mean>0.0</mean>
-                        <stddev>2e-4</stddev>
-                        <bias_mean>0.0000075</bias_mean>
-                        <bias_stddev>0.0000008</bias_stddev>
-                    </noise>
-                    </y>
-                    <z>
-                    <noise type="gaussian">
-                        <mean>0.0</mean>
-                        <stddev>2e-4</stddev>
-                        <bias_mean>0.0000075</bias_mean>
-                        <bias_stddev>0.0000008</bias_stddev>
-                    </noise>
-                    </z>
-                </angular_velocity>
-                <linear_acceleration>
-                    <x>
-                    <noise type="gaussian">
-                        <mean>0.0</mean>
-                        <stddev>1.7e-2</stddev>
-                        <bias_mean>0.1</bias_mean>
-                        <bias_stddev>0.001</bias_stddev>
-                    </noise>
-                    </x>
-                    <y>
-                    <noise type="gaussian">
-                        <mean>0.0</mean>
-                        <stddev>1.7e-2</stddev>
-                        <bias_mean>0.1</bias_mean>
-                        <bias_stddev>0.001</bias_stddev>
-                    </noise>
-                    </y>
-                    <z>
-                    <noise type="gaussian">
-                        <mean>0.0</mean>
-                        <stddev>1.7e-2</stddev>
-                        <bias_mean>0.1</bias_mean>
-                        <bias_stddev>0.001</bias_stddev>
-                    </noise>
-                    </z>
-                </linear_acceleration>
-            </imu>
-        </sensor> -->
-    </gazebo>
 </robot>

File: src/wro_ws/src/robot_description/urdf/ros2_control_bic.xacro (robot description, xacro)
@@ -8,5 +8,4 @@
             <param name="loop_rate">30</param>
             <param name="device">/dev/serial/by-id/usb-1a86_USB2.0-Ser_-if00-port0</param>
-            <!-- <param name="device">/dev/serial/by-path/pci-0000:00:14.0-usb-0:4:1.0-port0</param> -->
             <param name="baud_rate">9600</param>
             <param name="timeout_ms">1000</param>
